File: pcb/_autosave-micro.kicad_sch (KiCad schematic)
At the start: 16 parts, among them U1 ESP32-C6

Commit message: updated read me
Connections:
- net +3.3V: now also U1.40 (VDDA2)
- net GND: now also U1.41 (GND)
Other:
- note added: "ESP32-C6 needs power RC enable delay external SPI flash clock Matrix RF antenna Boot mode ESD"
- note removed: "ESP32-C6 needs power RC enable delay external SPI flash clock RF antenna Boot mode ESD"
Changed lines of the file:
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@@
 		)
 	)
-	(text "ESP32-C6 needs power \nRC enable delay \nexternal SPI flash \nclock \nRF antenna\nBoot mode\nESD"
+	(text "ESP32-C6 needs power \nRC enable delay \nexternal SPI flash \nclock \nMatrix\nRF antenna\nBoot mode\nESD"
 		(exclude_from_sim no)
 		(at 129.54 43.434 0)
@@
 	)
 	(junction
+		(at 142.24 67.31)
+		(diameter 0)
+		(color 0 0 0 0)
+	)
+	(junction
 		(at 152.4 74.93)
 		(diameter 0)
@@
 	(wire
 		(pts
+			(xy 147.32 138.43) (xy 147.32 133.35)
+		)
+		(stroke
+			(width 0)
+			(type default)
+		)
+	)
+	(wire
+		(pts
 			(xy 196.85 100.33) (xy 196.85 101.6)
 		)
@@
 	(wire
 		(pts
+			(xy 147.32 133.35) (xy 142.24 133.35)
+		)
+		(stroke
+			(width 0)
+			(type default)
+		)
+	)
+	(wire
+		(pts
 			(xy 226.06 118.11) (xy 232.41 118.11)
 		)
@@
 		(pts
 			(xy 55.88 80.01) (xy 63.5 80.01)
+		)
+		(stroke
+			(width 0)
+			(type default)
+		)
+	)
+	(wire
+		(pts
+			(xy 142.24 67.31) (xy 142.24 69.85)
 		)
 		(stroke
@@
 					(unit 1)
 				)
+			)
+		)
+	)
+	(symbol
+		(lib_id "power:GND")
+		(at 147.32 138.43 0)
+		(unit 1)
+		(exclude_from_sim no)
+		(in_bom yes)
+		(on_board yes)
+		(dnp no)
+		(fields_autoplaced yes)
+		(property "Reference" "#PWR08"
+			(at 147.32 144.78 0)
+			(effects
+				(font
+					(size 1.27 1.27)
+				)
+				(hide yes)
+			)
+		)
+		(property "Value" "GND"
+			(at 147.32 143.51 0)
+			(effects
+				(font
+					(size 1.27 1.27)
+				)
+			)
+		)
+		(property "Footprint" ""
+			(at 147.32 138.43 0)
+			(effects
+				(font
+					(size 1.27 1.27)
+				)
+				(hide yes)
+			)
+		)
+		(property "Datasheet" ""
+			(at 147.32 138.43 0)
+			(effects
+				(font
+					(size 1.27 1.27)
+				)
+				(hide yes)
+			)
+		)
+		(property "Description" "Power symbol creates a global label with name \"GND\" , ground"
+			(at 147.32 138.43 0)
+			(effects
+				(font
+					(size 1.27 1.27)
+				)
+				(hide yes)
+			)
+		)
+		(pin "1"
+		)
+		(instances
+			(project "60_keyboard"
+				(path "/60f4ab9d-718b-428d-904c-5042759d3860/a5dc5d45-cfa6-4235-a666-1339e0663470"
+					(reference "#PWR08")
+					(unit 1)
+				)
