File: pcb/60_keyboard.kicad_pcb (KiCad board)
At the start: 2 copper layers, 108 parts, among them SW1 SW_MX, SW10 SW_MX, SW11 SW_MX, SW12 SW_MX, SW13 SW_MX, SW14 SW_MX, SW15 SW_MX, SW16 SW_MX, SW17 SW_MX, SW18 SW_MX, SW19 SW_MX, SW2 SW_MX, SW20 SW_MX, SW21 SW_MX, SW22 SW_MX, SW23 SW_MX, SW24 SW_MX, SW25 SW_MX, SW26 SW_MX, SW27 SW_MX, SW28 SW_MX, SW29 SW_MX, SW3 SW_MX, SW30 SW_MX, SW31 SW_MX, SW32 SW_MX, SW33 SW_MX, SW34 SW_MX, SW35 SW_MX, SW36 SW_MX, SW37 SW_MX, SW38 SW_MX, SW39 SW_MX, SW4 SW_MX, SW40 SW_MX, SW41 SW_MX, SW42 SW_MX, SW43 SW_MX, SW44 SW_MX, SW45 SW_MX, SW46 SW_MX, SW47 SW_MX, SW48 SW_MX, SW49 SW_MX, SW5 SW_MX, SW50 SW_MX, SW51 SW_MX, SW52 SW_MX, SW53 SW_MX, SW54 SW_MX, SW6 SW_MX, SW7 SW_MX, SW8 SW_MX, SW9 SW_MX

Commit message: All Schematic Parts Added
Parts:
- added C1: 10u, Capacitor_SMD:C_0402_1005Metric_Pad0.74x0.62mm_HandSolder, F.Cu at (191.5, 62.3)
- added C10: 0.1u, Resistor_SMD:R_0402_1005Metric_Pad0.72x0.64mm_HandSolder, F.Cu at (186.4, 35.6)
- added C11: 10u, Resistor_SMD:R_0402_1005Metric_Pad0.72x0.64mm_HandSolder, F.Cu at (186.4, 37.6)
- added C12: 1u, Resistor_SMD:R_0402_1005Metric_Pad0.72x0.64mm_HandSolder, F.Cu at (186.4, 39.6)
- added C13: 1u, Capacitor_SMD:C_0402_1005Metric_Pad0.74x0.62mm_HandSolder, F.Cu at (198.3, 42.9)
- added C14: 14p, Resistor_SMD:R_0402_1005Metric_Pad0.72x0.64mm_HandSolder, F.Cu at (186.4, 41.6)
- added C15: 14p, Resistor_SMD:R_0402_1005Metric_Pad0.72x0.64mm_HandSolder, F.Cu at (186.4, 43.6)
- added C2: 10u, Capacitor_SMD:C_0402_1005Metric_Pad0.74x0.62mm_HandSolder, F.Cu at (191.5, 64.2)
- added C3: 0.1u, Resistor_SMD:R_0402_1005Metric_Pad0.72x0.64mm_HandSolder, F.Cu at (183.1, 35.6)
- added C4: 0.1u, Resistor_SMD:R_0402_1005Metric_Pad0.72x0.64mm_HandSolder, F.Cu at (183.1, 37.6)
- added C5: 1u, Resistor_SMD:R_0402_1005Metric_Pad0.72x0.64mm_HandSolder, F.Cu at (183.1, 39.6)
- added C6: 0.1u, Resistor_SMD:R_0402_1005Metric_Pad0.72x0.64mm_HandSolder, F.Cu at (183.1, 41.6)
- added C7: 10u, Resistor_SMD:R_0402_1005Metric_Pad0.72x0.64mm_HandSolder, F.Cu at (183.1, 43.6)
- added C8: 1u, Resistor_SMD:R_0402_1005Metric_Pad0.72x0.64mm_HandSolder, F.Cu at (183.1, 45.6)
- added C9: 0.1u, Resistor_SMD:R_0402_1005Metric_Pad0.72x0.64mm_HandSolder, F.Cu at (183.1, 47.6)
- added D100: BAV16W, Diode_SMD:D_SOD-123, F.Cu at (176.6, 29.5)
- added D101: BAV16W, Diode_SMD:D_SOD-123, F.Cu at (176.6, 32.9)
- added D102: BAV16W, Diode_SMD:D_SOD-123, F.Cu at (176.6, 36.2)
- added D103: BAV16W, Diode_SMD:D_SOD-123, F.Cu at (176.6, 39.6)
- added D104: BAV16W, Diode_SMD:D_SOD-123, F.Cu at (176.6, 42.9)
- added D105: BAV16W, Diode_SMD:D_SOD-123, F.Cu at (176.6, 46.3)
- added D106: BAV16W, Diode_SMD:D_SOD-123, F.Cu at (176.6, 49.6)
- added D107: BAV16W, Diode_SMD:D_SOD-123, F.Cu at (176.6, 53.0)
- added D108: BAV16W, Diode_SMD:D_SOD-123, F.Cu at (176.6, 56.3)
- added D55: BAV16W, Diode_SMD:D_SOD-123, F.Cu at (147.6, 29.5)
- added D56: BAV16W, Diode_SMD:D_SOD-123, F.Cu at (147.6, 32.9)
- added D57: BAV16W, Diode_SMD:D_SOD-123, F.Cu at (147.6, 36.2)
- added D58: BAV16W, Diode_SMD:D_SOD-123, F.Cu at (147.6, 39.6)
- added D59: BAV16W, Diode_SMD:D_SOD-123, F.Cu at (147.6, 42.9)
- added D60: BAV16W, Diode_SMD:D_SOD-123, F.Cu at (147.6, 46.3)
- added D61: BAV16W, Diode_SMD:D_SOD-123, F.Cu at (147.6, 49.6)
- added D62: BAV16W, Diode_SMD:D_SOD-123, F.Cu at (147.6, 53.0)
- added D63: BAV16W, Diode_SMD:D_SOD-123, F.Cu at (147.6, 56.3)
- added D64: BAV16W, Diode_SMD:D_SOD-123, F.Cu at (153.4, 29.5)
- added D65: BAV16W, Diode_SMD:D_SOD-123, F.Cu at (153.4, 32.9)
- added D66: BAV16W, Diode_SMD:D_SOD-123, F.Cu at (153.4, 36.2)
- added D67: BAV16W, Diode_SMD:D_SOD-123, F.Cu at (153.4, 39.6)
- added D68: BAV16W, Diode_SMD:D_SOD-123, F.Cu at (153.4, 42.9)
- added D69: BAV16W, Diode_SMD:D_SOD-123, F.Cu at (153.4, 46.3)
- added D70: BAV16W, Diode_SMD:D_SOD-123, F.Cu at (153.4, 49.6)
- added D71: BAV16W, Diode_SMD:D_SOD-123, F.Cu at (153.4, 53.0)
- added D72: BAV16W, Diode_SMD:D_SOD-123, F.Cu at (153.4, 56.3)
- added D73: BAV16W, Diode_SMD:D_SOD-123, F.Cu at (159.2, 29.5)
- added D74: BAV16W, Diode_SMD:D_SOD-123, F.Cu at (159.2, 32.9)
- added D75: BAV16W, Diode_SMD:D_SOD-123, F.Cu at (159.2, 36.2)
- added D76: BAV16W, Diode_SMD:D_SOD-123, F.Cu at (159.2, 39.6)
- added D77: BAV16W, Diode_SMD:D_SOD-123, F.Cu at (159.2, 42.9)
- added D78: BAV16W, Diode_SMD:D_SOD-123, F.Cu at (159.2, 46.3)
- added D79: BAV16W, Diode_SMD:D_SOD-123, F.Cu at (159.2, 49.6)
- added D80: BAV16W, Diode_SMD:D_SOD-123, F.Cu at (159.2, 53.0)
- added D81: BAV16W, Diode_SMD:D_SOD-123, F.Cu at (159.2, 56.3)
- added D82: BAV16W, Diode_SMD:D_SOD-123, F.Cu at (165.0, 29.5)
- added D83: BAV16W, Diode_SMD:D_SOD-123, F.Cu at (165.0, 32.9)
- added D84: BAV16W, Diode_SMD:D_SOD-123, F.Cu at (165.0, 36.2)
- added D85: BAV16W, Diode_SMD:D_SOD-123, F.Cu at (165.0, 39.6)
- added D86: BAV16W, Diode_SMD:D_SOD-123, F.Cu at (165.0, 42.9)
- added D87: BAV16W, Diode_SMD:D_SOD-123, F.Cu at (165.0, 46.3)
- added D88: BAV16W, Diode_SMD:D_SOD-123, F.Cu at (165.0, 49.6)
- added D89: BAV16W, Diode_SMD:D_SOD-123, F.Cu at (165.0, 53.0)
- added D90: BAV16W, Diode_SMD:D_SOD-123, F.Cu at (165.0, 56.3)
- added D91: BAV16W, Diode_SMD:D_SOD-123, F.Cu at (170.8, 29.5)
- added D92: BAV16W, Diode_SMD:D_SOD-123, F.Cu at (170.8, 32.9)
- added D93: BAV16W, Diode_SMD:D_SOD-123, F.Cu at (170.8, 36.2)
- added D94: BAV16W, Diode_SMD:D_SOD-123, F.Cu at (170.8, 39.6)
- added D95: BAV16W, Diode_SMD:D_SOD-123, F.Cu at (170.8, 42.9)
- added D96: BAV16W, Diode_SMD:D_SOD-123, F.Cu at (170.8, 46.3)
- added D97: BAV16W, Diode_SMD:D_SOD-123, F.Cu at (170.8, 49.6)
- added D98: BAV16W, Diode_SMD:D_SOD-123, F.Cu at (170.8, 53.0)
- added D99: BAV16W, Diode_SMD:D_SOD-123, F.Cu at (170.8, 56.3)
- added J2: USB_C_Receptacle_USB2.0_14P, Connector_USB:USB_C_Receptacle_HRO_TYPE-C-31-M-12, F.Cu at (187.3, 56.6)
- added L1: 2n, Inductor_SMD:L_0402_1005Metric_Pad0.77x0.64mm_HandSolder, F.Cu at (186.4, 45.6)
- added L2: 2n, Inductor_SMD:L_0402_1005Metric_Pad0.77x0.64mm_HandSolder, F.Cu at (186.4, 47.6)
- added R1: 5.1K, Resistor_SMD:R_0402_1005Metric_Pad0.72x0.64mm_HandSolder, F.Cu at (188.3, 62.3)
- added R2: 5.1K, Resistor_SMD:R_0402_1005Metric_Pad0.72x0.64mm_HandSolder, F.Cu at (188.3, 64.3)
- added R3: 10k, Resistor_SMD:R_0402_1005Metric_Pad0.72x0.64mm_HandSolder, F.Cu at (189.6, 35.6)
- added R4: 10k, Resistor_SMD:R_0402_1005Metric_Pad0.72x0.64mm_HandSolder, F.Cu at (189.6, 37.6)
- added R5: 10k, Resistor_SMD:R_0402_1005Metric_Pad0.72x0.64mm_HandSolder, F.Cu at (189.6, 39.6)
- added R6: 10k, Resistor_SMD:R_0402_1005Metric_Pad0.72x0.64mm_HandSolder, F.Cu at (189.6, 41.6)
- added SW1: SW_Nidec_CAS-120A1, Button_Switch_SMD:Nidec_Copal_CAS-120A, F.Cu at (194.0, 45.3)
- added SW100: SW_MX, Keyboard:CherryMX_1.00u, F.Cu at (136.3, 36.2)
- added SW101: SW_MX, Keyboard:CherryMX_1.00u, F.Cu at (136.3, 52.9)
- added SW102: SW_MX, Keyboard:CherryMX_1.00u, F.Cu at (136.3, 69.6)
- added SW103: SW_MX, Keyboard:CherryMX_1.00u, F.Cu at (136.3, 86.4)
- added SW104: SW_MX, Keyboard:CherryMX_1.00u, F.Cu at (136.3, 103.1)
- added SW105: SW_MX, Keyboard:CherryMX_1.50u, F.Cu at (136.3, 119.8)
- added SW106: SW_MX, Keyboard:CherryMX_1.50u, F.Cu at (136.3, 136.5)
- added SW107: SW_MX, Keyboard:CherryMX_3.00u, F.Cu at (136.3, 153.2)
- added SW108: SW_MX, Keyboard:CherryMX_1.50u, F.Cu at (136.3, 170.0)
- added SW55: SW_MX, Keyboard:CherryMX_1.50u, F.Cu at (52.7, 36.2)
- added SW56: SW_MX, Keyboard:CherryMX_1.50u, F.Cu at (52.7, 52.9)
- added SW57: SW_MX, Keyboard:CherryMX_1.50u, F.Cu at (52.7, 69.6)
- added SW58: SW_MX, Keyboard:CherryMX_1.50u, F.Cu at (52.7, 86.4)
- added SW59: SW_MX, Keyboard:CherryMX_1.00u, F.Cu at (52.7, 103.1)
- added SW60: SW_MX, Keyboard:CherryMX_1.00u, F.Cu at (52.7, 119.8)
- added SW61: SW_MX, Keyboard:CherryMX_1.00u, F.Cu at (52.7, 136.5)
- added SW62: SW_MX, Keyboard:CherryMX_1.00u, F.Cu at (52.7, 153.2)
- added SW63: SW_MX, Keyboard:CherryMX_1.00u, F.Cu at (52.7, 170.0)
- added SW64: SW_MX, Keyboard:CherryMX_1.00u, F.Cu at (69.5, 36.2)
- added SW65: SW_MX, Keyboard:CherryMX_1.00u, F.Cu at (69.5, 52.9)
- added SW66: SW_MX, Keyboard:CherryMX_1.00u, F.Cu at (69.5, 69.6)
- added SW67: SW_MX, Keyboard:CherryMX_1.00u, F.Cu at (69.5, 86.4)
- added SW68: SW_MX, Keyboard:CherryMX_1.00u, F.Cu at (69.5, 103.1)
- added SW69: SW_MX, Keyboard:CherryMX_1.00u, F.Cu at (69.5, 119.8)
- added SW70: SW_MX, Keyboard:CherryMX_1.00u, F.Cu at (69.5, 136.5)
- added SW71: SW_MX, Keyboard:CherryMX_1.00u, F.Cu at (69.5, 153.2)
- added SW72: SW_MX, Keyboard:CherryMX_1.00u, F.Cu at (69.5, 170.0)
- added SW73: SW_MX, Keyboard:CherryMX_1.00u, F.Cu at (86.2, 36.2)
- added SW74: SW_MX, Keyboard:CherryMX_1.00u, F.Cu at (86.2, 52.9)
- added SW75: SW_MX, Keyboard:CherryMX_1.00u, F.Cu at (86.2, 69.6)
- added SW76: SW_MX, Keyboard:CherryMX_1.00u, F.Cu at (86.2, 86.4)
- added SW77: SW_MX, Keyboard:CherryMX_1.00u, F.Cu at (86.2, 103.1)
- added SW78: SW_MX, Keyboard:CherryMX_1.00u, F.Cu at (86.2, 119.8)
- added SW79: SW_MX, Keyboard:CherryMX_1.00u, F.Cu at (86.2, 136.5)
- added SW80: SW_MX, Keyboard:CherryMX_1.00u, F.Cu at (86.2, 153.2)
- added SW81: SW_MX, Keyboard:CherryMX_1.00u, F.Cu at (86.2, 170.0)
- added SW82: SW_MX, Keyboard:CherryMX_1.00u, F.Cu at (102.9, 36.2)
- added SW83: SW_MX, Keyboard:CherryMX_1.00u, F.Cu at (102.9, 52.9)
- added SW84: SW_MX, Keyboard:CherryMX_1.00u, F.Cu at (102.9, 69.6)
- added SW85: SW_MX, Keyboard:CherryMX_1.00u, F.Cu at (102.9, 86.4)
- added SW86: SW_MX, Keyboard:CherryMX_1.00u, F.Cu at (102.9, 103.1)
- added SW87: SW_MX, Keyboard:CherryMX_1.00u, F.Cu at (102.9, 119.8)
- added SW88: SW_MX, Keyboard:CherryMX_1.00u, F.Cu at (102.9, 136.5)
- added SW89: SW_MX, Keyboard:CherryMX_1.00u, F.Cu at (102.9, 153.2)
- added SW90: SW_MX, Keyboard:CherryMX_1.00u, F.Cu at (102.9, 170.0)
- added SW91: SW_MX, Keyboard:CherryMX_1.00u, F.Cu at (119.6, 36.2)
- added SW92: SW_MX, Keyboard:CherryMX_1.00u, F.Cu at (119.6, 52.9)
- added SW93: SW_MX, Keyboard:CherryMX_1.00u, F.Cu at (119.6, 69.6)
- added SW94: SW_MX, Keyboard:CherryMX_1.00u, F.Cu at (119.6, 86.4)
- added SW95: SW_MX, Keyboard:CherryMX_1.00u, F.Cu at (119.6, 103.1)
- added SW96: SW_MX, Keyboard:CherryMX_1.00u, F.Cu at (119.6, 119.8)
- added SW97: SW_MX, Keyboard:CherryMX_1.00u, F.Cu at (119.6, 136.5)
- added SW98: SW_MX, Keyboard:CherryMX_1.00u, F.Cu at (119.6, 153.2)
- added SW99: SW_MX, Keyboard:CherryMX_1.00u, F.Cu at (119.6, 170.0)
- added U1: ESP32-C6, ESP32:QFN40P500X500X90-41N, F.Cu at (195.5, 38.2)
- added U2: XC6220B331MR, Package_TO_SOT_SMD:SOT-23-5, F.Cu at (184.0, 63.7)
- added U3: ~, ESP32:SOIC127P790X216-8N, F.Cu at (187.4, 31.2)
- added Y1: 7M40000049, ESP32:XTAL_7M40000049, F.Cu at (195.5, 30.4)
- moved D1 1652.1 mm to (431.8, 24.1)
- moved D10 1652.1 mm to (437.6, 24.1)
- moved D11 1652.1 mm to (437.6, 27.4)
- moved D12 1652.1 mm to (437.6, 30.8)
- moved D13 1652.1 mm to (437.6, 34.1)
- moved D14 1652.1 mm to (437.6, 37.5)
- moved D15 1652.1 mm to (437.6, 40.8)
- moved D16 1652.1 mm to (437.6, 44.2)
- moved D17 1652.1 mm to (437.6, 47.5)
- moved D18 1652.1 mm to (437.6, 50.9)
- moved D2 1652.1 mm to (431.8, 27.4)
- moved D28 1652.1 mm to (449.2, 24.1)
- moved D29 1652.1 mm to (449.2, 27.4)
- moved D3 1652.1 mm to (431.8, 30.8)
- moved D30 1652.1 mm to (449.2, 30.8)
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