File: pcb/60_keyboard.kicad_pcb (KiCad board)
At the start: 2 copper layers, 247 x 100 mm, 144 parts, among them J2 USB_C_Receptacle_USB2.0_14P, SW1 SW_Nidec_CAS-120A1, SW100 SW_MX, SW101 SW_MX, SW102 SW_MX, SW103 SW_MX, SW104 SW_MX, SW105 SW_MX, SW106 SW_MX, SW107 SW_MX, SW108 SW_MX, SW55 SW_MX, SW56 SW_MX, SW57 SW_MX, SW58 SW_MX, SW59 SW_MX, SW60 SW_MX, SW61 SW_MX, SW62 SW_MX, SW63 SW_MX, SW64 SW_MX, SW65 SW_MX, SW66 SW_MX, SW67 SW_MX, SW68 SW_MX, SW69 SW_MX, SW70 SW_MX, SW71 SW_MX, SW72 SW_MX, SW73 SW_MX, SW74 SW_MX, SW75 SW_MX, SW76 SW_MX, SW77 SW_MX, SW78 SW_MX, SW79 SW_MX, SW80 SW_MX, SW81 SW_MX, SW82 SW_MX, SW83 SW_MX, SW84 SW_MX, SW85 SW_MX, SW86 SW_MX, SW87 SW_MX, SW88 SW_MX, SW89 SW_MX, SW90 SW_MX, SW91 SW_MX, SW92 SW_MX, SW93 SW_MX, SW94 SW_MX, SW95 SW_MX, SW96 SW_MX, SW97 SW_MX, SW98 SW_MX, SW99 SW_MX, U1 ESP32-C6, U2 XC6220B331MR, Y1 7M40000049

Commit message: Finished board, with maybe some cleanup needed
Parts:
- removed D2, D3: D_TVS, Diode_SMD:D_SOD-123
- removed J2: USB_C_Receptacle_USB2.0_14P, Connector_USB:USB_C_Receptacle_HRO_TYPE-C-31-M-12
- added J1: USB_C_Receptacle_USB2.0_16P, Connector_USB:USB_C_Receptacle_HRO_TYPE-C-31-M-12, B.Cu at (236.0, 12.5)
- C1, C10, C11, C12, C13, C14, C15, C2, C3, C4, C5, C6, C7, C8, C9, L1, R2, R3, R7, R8, U1, U2, U3, Y1: moved to B.Cu
- D1, D5: footprint Diode_SMD:D_SOD-123 -> Diode_SMD:D_SOD-323_HandSoldering; moved to B.Cu
- D4: footprint Diode_SMD:D_SOD-123 -> Diode_SMD:D_SOD-323_HandSoldering
- L2: value 2n -> 24n; moved to B.Cu
- moved D5 142.7 mm to (234.2, 20.2), turned to 180 degrees
- moved R2 142.6 mm to (233.2, 18.5), turned to 180 degrees
- moved D4 141.1 mm to (234.5, 18.5), turned to 180 degrees
- moved R1 140.6 mm to (239.0, 18.5)
- moved C1 140.6 mm to (239.0, 18.5)
- moved U2 139.5 mm to (239.5, 21.2), turned to -90 degrees
- moved C2 139.3 mm to (237.2, 21.8), turned to 90 degrees
- moved D1 133.3 mm to (242.5, 17.0), turned to 90 degrees
- moved SW1 129.0 mm to (221.2, 13.1), turned to 90 degrees
- moved R6 120.0 mm to (227.0, 13.8), turned to 90 degrees
- moved R5 118.1 mm to (225.8, 13.8), turned to 90 degrees
- moved R8 114.3 mm to (235.5, 23.2), turned to 90 degrees
- moved C13 113.9 mm to (228.8, 31.5), turned to 90 degrees
- moved R7 112.3 mm to (234.5, 23.2), turned to -90 degrees
- moved U3 110.4 mm to (242.7, 31.8), turned to -90 degrees
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Connections:
- C3 pad 1: Net-(U1-VDDPST1) -> +3.3V
- C4 pad 1: Net-(U1-VDDPST1) -> +3.3V
- D60 pad 1: unconnected-(D60-K-Pad1) -> Col 2
- D69 pad 1: unconnected-(D69-K-Pad1) -> Col 4
- D73 pad 1: unconnected-(D73-K-Pad1) -> Col 5
- D74 pad 1: unconnected-(D74-K-Pad1) -> Col 5
- D75 pad 1: unconnected-(D75-K-Pad1) -> Col 5
- D76 pad 1: unconnected-(D76-K-Pad1) -> Col 5
- U1 pad 10: unconnected-(U1-GPIO4/MTMS-Pad10) -> Col 5
- U1 pad 11: unconnected-(U1-GPIO5/MTDI-Pad11) -> Col 6
- U1 pad 12: unconnected-(U1-GPIO6/MTCK-Pad12) -> Col 7
- U1 pad 13: unconnected-(U1-GPIO7/MTDO-Pad13) -> Col 8
- U1 pad 16: unconnected-(U1-GPIO10-Pad16) -> Col 9
- U1 pad 17: unconnected-(U1-GPIO11-Pad17) -> Col 10
- U1 pad 27: unconnected-(U1-GPIO15-Pad27) -> Col 11
- U1 pad 28: Net-(U1-VDDPST1) -> +3.3V
- U1 pad 29: unconnected-(U1-U0TXD/GPIO16-Pad29) -> Col 12
- U1 pad 32: unconnected-(U1-SDIO_CLK/GPIO19-Pad32) -> Row 1
- U1 pad 33: unconnected-(U1-SDIO_DATA0/GPIO20-Pad33) -> Row 2
- U1 pad 34: unconnected-(U1-SDIO_DATA1/GPIO21-Pad34) -> Row 3
- U1 pad 35: unconnected-(U1-SDIO_DATA2/GPIO22-Pad35) -> Row 4
- U1 pad 36: unconnected-(U1-SDIO_DATA3/GPIO23-Pad36) -> Row 5
- U1 pad 5: Net-(U1-VDDPST1) -> +3.3V
- U1 pad 6: unconnected-(U1-GPIO0/XTAL_32K_P-Pad6) -> Col 1
- U1 pad 7: unconnected-(U1-GPIO1/XTAL_32K_N-Pad7) -> Col 2
- U1 pad 8: unconnected-(U1-GPIO2-Pad8) -> Col 3
- U1 pad 9: unconnected-(U1-GPIO3-Pad9) -> Col 4
Routing:
- net Col 1: track 0.00 -> 263.1 mm, vias 0 -> 2
- net Col 3: track 0.00 -> 244.6 mm, vias 0 -> 2
- net Col 2: track 0.00 -> 240.7 mm, vias 0 -> 2
- net Col 4: track 0.00 -> 226.0 mm, vias 0 -> 2
- net Col 5: track 0.00 -> 206.5 mm, vias 0 -> 2
- net Col 7: track 0.00 -> 170.0 mm, vias 0 -> 2
- net Col 6: track 0.00 -> 166.7 mm, vias 0 -> 2
- net Col 9: track 0.00 -> 136.2 mm, vias 0 -> 2
- net Col 8: track 0.00 -> 130.7 mm, vias 0 -> 2
- net Row 5: track 133.0 -> 251.3 mm, vias 0 -> 1
- net Col 10: track 0.00 -> 117.3 mm, vias 0 -> 2
- net +3.3V: track 0.00 -> 88.8 mm, vias 0 -> 11
- net Col 11: track 0.00 -> 87.9 mm, vias 0 -> 2
- net Col 12: track 0.00 -> 85.6 mm
- net Row 4: track 218.5 -> 281.0 mm, vias 0 -> 1
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- added copper zone on B.Cu, net GND
- added copper zone on F.Cu, net GND

Commit message: board almost finished
Parts:
- C10, C11, C12, C14, C15, C3, C4, C5, C6, C7, C8, C9: footprint Resistor_SMD:R_0402_1005Metric_Pad0.72x0.64mm_HandSolder -> Capacitor_SMD:C_0402_1005Metric_Pad0.74x0.62mm_HandSolder
- D4, R1, R4, R5, R6, SW1: moved to B.Cu
- SW100, SW101, SW102, SW103, SW104, SW59, SW60, SW61, SW62, SW63, SW64, SW65, SW66, SW67, SW68, SW69, SW70, SW71, SW72, SW73, SW74, SW75, SW76, SW77, SW78, SW79, SW80, SW81, SW82, SW83, SW84, SW85, SW87, SW88, SW89, SW90, SW91, SW92, SW93, SW94, SW95, SW96, SW97, SW98, SW99: footprint Keyboard:CherryMX_1.00u -> Keyboard:Hot_Swap; moved to B.Cu
- SW105, SW106, SW107, SW108, SW55, SW56, SW57, SW58: footprint Keyboard:CherryMX_1.50u -> Keyboard:Hot_Swap; moved to B.Cu
- SW86: footprint Keyboard:CherryMX_3.00u -> Keyboard:Hot_Swap; moved to B.Cu
- moved R4 7.07 mm to (246.2, 29.5)
- moved U2 4.55 mm to (238.2, 25.6)
- moved C2 4.42 mm to (240.5, 24.8)
- moved D105 3.25 mm to (251.5, 29.8), turned to 0 degrees
- moved R1 3.25 mm to (242.2, 18.5)
- moved R6 3.02 mm to (229.8, 15.0)
- moved SW1 2.93 mm to (224.0, 14.1)
- moved R5 2.80 mm to (228.2, 15.0)
- moved C14 1.91 mm to (232.2, 38.0)
- moved R2 1.75 mm to (233.2, 20.2)
- moved Y1 1.63 mm to (235.0, 38.6)
- moved C15 1.57 mm to (237.8, 37.8)
- moved D5 1.50 mm to (234.2, 21.8)
- moved D1 1.27 mm to (242.8, 15.8)
- moved R7 1.03 mm to (234.8, 24.2)
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Routing:
- net Net-(D105-A): track 8.89 -> 20.7 mm
- net Net-(SW1-A): track 22.3 -> 32.5 mm, vias 1 -> 0
- net SPI3.3: track 9.94 -> 17.3 mm, vias 1 -> 0
- net ~CS: track 6.56 -> 12.6 mm, vias 1 -> 0
- net Vin: track 15.6 -> 21.4 mm
- net Net-(D86-A): track 8.43 -> 12.1 mm
- net Net-(D76-A): track 8.43 -> 12.1 mm
- net Net-(D71-A): track 8.48 -> 12.1 mm
- net Net-(D55-A): track 8.48 -> 12.1 mm
- net Net-(D99-A): track 8.43 -> 12.0 mm
- net Net-(D83-A): track 8.68 -> 12.2 mm
- net Net-(D65-A): track 8.68 -> 12.2 mm
- net Net-(D107-A): track 8.43 -> 12.0 mm
- net Net-(D75-A): track 8.48 -> 11.9 mm
- net Net-(D108-A): track 8.37 -> 11.8 mm
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
Commit message: Finished board
Routing:
- net Row 1: track 246.5 -> 272.5 mm, vias 1 -> 12
- net Row 3: track 261.1 -> 286.3 mm, vias 1 -> 12
- net Row 2: track 236.0 -> 254.0 mm, vias 1 -> 12
- net Col 1: track 263.1 -> 279.7 mm
- net Col 3: track 244.6 -> 260.4 mm
- net Col 5: track 206.5 -> 222.3 mm
- net Col 4: track 226.0 -> 241.4 mm
- net Col 7: track 170.0 -> 185.2 mm
- net Col 10: track 117.3 -> 132.4 mm
- net Col 9: track 136.2 -> 150.9 mm
- net Col 12: track 85.6 -> 98.2 mm
- net Col 8: track 130.7 -> 142.7 mm
- net Col 6: track 166.7 -> 178.5 mm
- net Col 2: track 240.7 -> 252.1 mm
- net Col 11: track 89.1 -> 97.3 mm
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
Commit message: Finished board
Parts:
- moved C15 0.50 mm to (237.8, 38.2)
Routing:
- net Row 4: track 283.2 -> 306.7 mm, vias 2 -> 13
- net Row 5: track 256.0 -> 264.4 mm, vias 2 -> 7
- net Row 1: track 272.5 -> 275.7 mm, vias 12 -> 13
- net Row 3: track 286.3 -> 289.0 mm, vias 12 -> 13
- net Row 2: track 254.0 -> 256.7 mm, vias 12 -> 13
- net XTAL_N: track 7.13 -> 9.04 mm
- net Col 3: track 260.4 -> 261.0 mm
- net GND: vias 39 -> 40

Commit message: Finished for day
Parts:
- added REF**: Stabilizer_Cherry_MX_3.00u, Keyboard:Stabilizer_Cherry_MX_3.00u, F.Cu at (148.0, 100.5)
Routing:
- net Row 5: track 264.4 -> 267.1 mm
Other:
- board size 247 x 100 mm -> 247 x 102.5 mm

Commit message: ordered board
Parts:
- moved R1 3.05 mm to (244.0, 16.0), turned to 90 degrees
- moved D1 0.79 mm to (242.5, 15.0)
Routing:
- net Net-(J1-CC2): track 5.48 -> 8.61 mm
- net +3.3V: track 89.4 -> 90.1 mm
