File: pcb/_autosave-60_keyboard.kicad_pcb (KiCad board)
At the start: 2 copper layers, 247 x 100 mm, 144 parts, among them J2 USB_C_Receptacle_USB2.0_14P, SW1 SW_Nidec_CAS-120A1, SW100 SW_MX, SW101 SW_MX, SW102 SW_MX, SW103 SW_MX, SW104 SW_MX, SW105 SW_MX, SW106 SW_MX, SW107 SW_MX, SW108 SW_MX, SW55 SW_MX, SW56 SW_MX, SW57 SW_MX, SW58 SW_MX, SW59 SW_MX, SW60 SW_MX, SW61 SW_MX, SW62 SW_MX, SW63 SW_MX, SW64 SW_MX, SW65 SW_MX, SW66 SW_MX, SW67 SW_MX, SW68 SW_MX, SW69 SW_MX, SW70 SW_MX, SW71 SW_MX, SW72 SW_MX, SW73 SW_MX, SW74 SW_MX, SW75 SW_MX, SW76 SW_MX, SW77 SW_MX, SW78 SW_MX, SW79 SW_MX, SW80 SW_MX, SW81 SW_MX, SW82 SW_MX, SW83 SW_MX, SW84 SW_MX, SW85 SW_MX, SW86 SW_MX, SW87 SW_MX, SW88 SW_MX, SW89 SW_MX, SW90 SW_MX, SW91 SW_MX, SW92 SW_MX, SW93 SW_MX, SW94 SW_MX, SW95 SW_MX, SW96 SW_MX, SW97 SW_MX, SW98 SW_MX, SW99 SW_MX, U1 ESP32-C6, U2 XC6220B331MR, Y1 7M40000049

Commit message: Schematic finalized and general layout completed
Routing:
- net (no net): vias 0 -> 4
Changed lines of the file:
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@@
 	)
 	(setup
+		(stackup
+			(layer "F.SilkS"
+				(type "Top Silk Screen")
+			)
+			(layer "F.Paste"
+				(type "Top Solder Paste")
+			)
+			(layer "F.Mask"
+				(type "Top Solder Mask")
+				(thickness 0.01)
+			)
+			(layer "F.Cu"
+				(type "copper")
+				(thickness 0.035)
+			)
+			(layer "dielectric 1"
+				(type "core")
+				(thickness 1.51)
+				(material "FR4")
+				(epsilon_r 4.5)
+				(loss_tangent 0.02)
+			)
+			(layer "B.Cu"
+				(type "copper")
+				(thickness 0.035)
+			)
+			(layer "B.Mask"
+				(type "Bottom Solder Mask")
+				(thickness 0.01)
+			)
+			(layer "B.Paste"
+				(type "Bottom Solder Paste")
+			)
+			(layer "B.SilkS"
+				(type "Bottom Silk Screen")
+			)
+			(copper_finish "None")
+			(dielectric_constraints no)
+		)
 		(pad_to_mask_clearance 0)
 		(allow_soldermask_bridges_in_footprints no)
@@
 		(layer "Edge.Cuts")
 	)
+	(via
+		(at 20 105)
+		(size 5.5)
+		(drill 3.2)
+		(layers "F.Cu" "B.Cu")
+		(tenting none)
+		(net 0)
+	)
+	(via
+		(at 257 105)
+		(size 5.5)
+		(drill 3.2)
+		(layers "F.Cu" "B.Cu")
+		(tenting none)
+		(net 0)
+	)
+	(via
+		(at 257 15)
+		(size 5.5)
+		(drill 3.2)
+		(layers "F.Cu" "B.Cu")
+		(tenting none)
+		(net 0)
+	)
+	(via
+		(at 20 15)
+		(size 5.5)
+		(drill 3.2)
+		(layers "F.Cu" "B.Cu")
+		(tenting none)
+		(net 0)
+	)
 	(segment
