File: pcb/_autosave-60_keyboard.kicad_pcb (KiCad board)
At the start: 2 copper layers, 247 x 100 mm, 142 parts, among them J1 USB_C_Receptacle_USB2.0_16P, SW1 SW_Nidec_CAS-120A1, SW100 SW_MX, SW101 SW_MX, SW102 SW_MX, SW103 SW_MX, SW104 SW_MX, SW105 SW_MX, SW106 SW_MX, SW107 SW_MX, SW108 SW_MX, SW55 SW_MX, SW56 SW_MX, SW57 SW_MX, SW58 SW_MX, SW59 SW_MX, SW60 SW_MX, SW61 SW_MX, SW62 SW_MX, SW63 SW_MX, SW64 SW_MX, SW65 SW_MX, SW66 SW_MX, SW67 SW_MX, SW68 SW_MX, SW69 SW_MX, SW70 SW_MX, SW71 SW_MX, SW72 SW_MX, SW73 SW_MX, SW74 SW_MX, SW75 SW_MX, SW76 SW_MX, SW77 SW_MX, SW78 SW_MX, SW79 SW_MX, SW80 SW_MX, SW81 SW_MX, SW82 SW_MX, SW83 SW_MX, SW84 SW_MX, SW85 SW_MX, SW86 SW_MX, SW87 SW_MX, SW88 SW_MX, SW89 SW_MX, SW90 SW_MX, SW91 SW_MX, SW92 SW_MX, SW93 SW_MX, SW94 SW_MX, SW95 SW_MX, SW96 SW_MX, SW97 SW_MX, SW98 SW_MX, SW99 SW_MX, U1 ESP32-C6, U2 XC6220B331MR, Y1 7M40000049

Commit message: board almost finished
Parts:
- D4, R1, R4, R5, R6, SW1: moved to B.Cu
- SW100, SW101, SW102, SW103, SW104, SW59, SW60, SW61, SW62, SW63, SW64, SW65, SW66, SW67, SW68, SW69, SW70, SW71, SW72, SW73, SW74, SW75, SW76, SW77, SW78, SW79, SW80, SW81, SW82, SW83, SW84, SW85, SW87, SW88, SW89, SW90, SW91, SW92, SW93, SW94, SW95, SW96, SW97, SW98, SW99: footprint Keyboard:CherryMX_1.00u -> Keyboard:Hot_Swap; moved to B.Cu
- SW105, SW106, SW107, SW108, SW55, SW56, SW57, SW58: footprint Keyboard:CherryMX_1.50u -> Keyboard:Hot_Swap; moved to B.Cu
- SW86: footprint Keyboard:CherryMX_3.00u -> Keyboard:Hot_Swap; moved to B.Cu
- moved R4 7.07 mm to (246.2, 29.5)
- moved U2 4.55 mm to (238.2, 25.6)
- moved C2 4.42 mm to (240.5, 24.8)
- moved D105 3.25 mm to (251.5, 29.8), turned to 0 degrees
- moved R1 3.25 mm to (242.2, 18.5)
- moved R6 3.02 mm to (229.8, 15.0)
- moved SW1 2.93 mm to (224.0, 14.1)
- moved R5 2.80 mm to (228.2, 15.0)
- moved C14 1.91 mm to (232.2, 38.0)
- moved R2 1.75 mm to (233.2, 20.2)
- moved Y1 1.63 mm to (235.0, 38.6)
- moved C15 1.57 mm to (237.8, 37.8)
- moved D5 1.50 mm to (234.2, 21.8)
- moved D1 1.27 mm to (242.8, 15.8)
- moved R7 1.03 mm to (234.8, 24.2)
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Routing:
- net Row 1: track 246.3 -> 272.5 mm, vias 1 -> 12
- net Net-(D105-A): track 8.89 -> 20.3 mm
- net Net-(SW1-A): track 22.3 -> 32.5 mm, vias 1 -> 0
- net SPI3.3: track 9.94 -> 17.3 mm, vias 1 -> 0
- net ~CS: track 6.56 -> 12.6 mm, vias 1 -> 0
- net Vin: track 15.6 -> 21.4 mm
- net Net-(D86-A): track 8.43 -> 12.1 mm
- net Net-(D76-A): track 8.43 -> 12.1 mm
- net Net-(D71-A): track 8.48 -> 12.1 mm
- net Net-(D55-A): track 8.48 -> 12.1 mm
- net Net-(D99-A): track 8.43 -> 12.0 mm
- net Net-(D83-A): track 8.68 -> 12.2 mm
- net Net-(D65-A): track 8.68 -> 12.2 mm
- net Net-(D107-A): track 8.43 -> 12.0 mm
- net Net-(D75-A): track 8.48 -> 11.9 mm
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
Commit message: Finished board
Routing:
- net Row 3: track 261.1 -> 289.0 mm, vias 2 -> 13
- net Row 4: track 281.2 -> 306.7 mm, vias 2 -> 13
- net Row 2: track 236.0 -> 254.0 mm, vias 2 -> 12
- net Col 1: track 263.1 -> 279.7 mm
- net Col 3: track 244.6 -> 261.0 mm
- net Col 5: track 206.5 -> 222.3 mm
- net Col 4: track 226.0 -> 241.4 mm
- net Col 7: track 170.0 -> 185.2 mm
- net Col 10: track 117.3 -> 132.4 mm
- net Col 9: track 136.2 -> 150.9 mm
- net Row 5: track 251.5 -> 264.4 mm, vias 2 -> 7
- net Col 12: track 85.6 -> 98.2 mm
- net Col 8: track 130.7 -> 142.7 mm
- net Col 6: track 166.7 -> 178.5 mm
- net Col 2: track 240.7 -> 252.1 mm
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