File: pcb/micro.kicad_sch (KiCad schematic)
At the start: 16 parts, among them U1 ESP32-C6

Commit message: All Schematic Parts Added
Parts:
- added C14, C15: 14p, Resistor_SMD:R_0402_1005Metric_Pad0.72x0.64mm_HandSolder, symbol Device:C
- added L2: 2n, Inductor_SMD:L_0402_1005Metric_Pad0.77x0.64mm_HandSolder, symbol Device:L
- added R5, R6: 10k, Resistor_SMD:R_0402_1005Metric_Pad0.72x0.64mm_HandSolder, symbol Device:R
- added SW1: SW_Nidec_CAS-120A1, Button_Switch_SMD:Nidec_Copal_CAS-120A, symbol Switch:SW_Nidec_CAS-120A1
- added Y1: 7M40000049, ESP32:XTAL_7M40000049, symbol ESP32:7M40000049
Connections:
- net +3.3V: now also U1.40 (VDDA2), SW1.2 (B)
- net GND: now also U1.41 (GND), C14.2, C15.2, R5.2, R6.2, Y1.2 (GND), Y1.4 (GND_)
- net at U1.14 (GPIO8): now also R5.1, SW1.1 (C)
- net at U1.15 (GPIO9): now also R6.1, SW1.3 (A)
- net XTAL_N: now reaches U1.38 (XTAL_N)
- net XTAL_N: now also C15.1, Y1.3
- net XTAL_P: now reaches U1.39 (XTAL_P)
- net XTAL_P: now also L2.1
- new net: C14.1, L2.2, Y1.1
Other:
- note added: "CL is 9pF. If stray is estimated as 2pF Caps can be 7*2 for 14pF"
- note added: "ESD USB"
- note removed: "ESP32-C6 needs power RC enable delay external SPI flash clock RF antenna Boot mode ESD"

Commit message: Schematic finalized and general layout completed
Parts:
- added R7, R8: 22, Resistor_SMD:R_0402_1005Metric_Pad0.72x0.64mm_HandSolder, symbol Device:R
Connections:
- net D+: now also R8.2; no longer U1.19 (USB_D+/GPIO13)
- net D-: now also R7.1; no longer U1.18 (USB_D-/GPIO12)
- new net: R7.2, U1.18 (USB_D-/GPIO12)
- new net: R8.1, U1.19 (USB_D+/GPIO13)
Changed lines of the file:
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@@
 	(wire
 		(pts
-			(xy 142.24 87.63) (xy 148.59 87.63)
+			(xy 162.56 90.17) (xy 165.1 90.17)
 		)
 		(stroke
@@
 	(wire
 		(pts
+			(xy 142.24 87.63) (xy 144.78 87.63)
+		)
+		(stroke
+			(width 0)
+			(type default)
+		)
+	)
+	(wire
+		(pts
 			(xy 54.61 115.57) (xy 54.61 120.65)
 		)
@@
 	(wire
 		(pts
-			(xy 142.24 90.17) (xy 148.59 90.17)
-		)
-		(stroke
-			(width 0)
-			(type default)
-		)
-	)
-	(wire
-		(pts
 			(xy 113.03 176.53) (xy 97.79 176.53)
 		)
@@
 	(wire
 		(pts
+			(xy 142.24 90.17) (xy 154.94 90.17)
+		)
+		(stroke
+			(width 0)
+			(type default)
+		)
+	)
+	(wire
+		(pts
 			(xy 142.24 62.23) (xy 142.24 64.77)
 		)
@@
 	(wire
 		(pts
+			(xy 152.4 87.63) (xy 165.1 87.63)
+		)
+		(stroke
+			(width 0)
+			(type default)
+		)
+	)
+	(wire
+		(pts
 			(xy 76.2 85.09) (xy 81.28 85.09)
 		)
@@
 	(global_label "D+"
 		(shape input)
-		(at 148.59 90.17 0)
+		(at 165.1 90.17 0)
 		(fields_autoplaced yes)
 		(effects
@@
 		)
 		(property "Intersheetrefs" "${INTERSHEET_REFS}"
-			(at 154.4176 90.17 0)
+			(at 170.9276 90.17 0)
 			(effects
 				(font
@@
 	(global_label "D-"
 		(shape input)
-		(at 148.59 87.63 0)
+		(at 165.1 87.63 0)
 		(fields_autoplaced yes)
 		(effects
@@
 		)
 		(property "Intersheetrefs" "${INTERSHEET_REFS}"
-			(at 154.4176 87.63 0)
+			(at 170.9276 87.63 0)
 			(effects
 				(font
@@
 	)
 	(symbol
+		(lib_id "Device:R")
+		(at 148.59 87.63 270)
+		(unit 1)
+		(exclude_from_sim no)
+		(in_bom yes)
+		(on_board yes)
+		(dnp no)
+		(property "Reference" "R7"
+			(at 148.59 82.804 90)
+			(effects
+				(font
+					(size 1.27 1.27)
+				)
+			)
+		)
+		(property "Value" "22"
+			(at 148.59 85.344 90)
+			(effects
+				(font
+					(size 1.27 1.27)
+				)
+			)
+		)
+		(property "Footprint" "Resistor_SMD:R_0402_1005Metric_Pad0.72x0.64mm_HandSolder"
+			(at 148.59 85.852 90)
+			(effects
+				(font
+					(size 1.27 1.27)
+				)
+				(hide yes)
+			)
+		)
+		(property "Datasheet" "~"
+			(at 148.59 87.63 0)
+			(effects
+				(font
+					(size 1.27 1.27)
+				)
+				(hide yes)
+			)
+		)
+		(property "Description" "Resistor"
+			(at 148.59 87.63 0)
+			(effects
+				(font
+					(size 1.27 1.27)
+				)
+				(hide yes)
+			)
+		)
+		(pin "2"
+		)
+		(pin "1"
+		)
+		(instances
+			(project "60_keyboard"
+				(path "/60f4ab9d-718b-428d-904c-5042759d3860/a5dc5d45-cfa6-4235-a666-1339e0663470"
+					(reference "R7")
+					(unit 1)
+				)
+			)
+		)
+	)
+	(symbol
 		(lib_id "Device:C")
 		(at 259.08 66.04 0)
@@
 					(unit 1)
 				)
+			)
+		)
+	)
+	(symbol
+		(lib_id "Device:R")
+		(at 158.75 90.17 90)
+		(unit 1)
+		(exclude_from_sim no)
+		(in_bom yes)
+		(on_board yes)
+		(dnp no)
+		(property "Reference" "R8"
+			(at 158.496 92.964 90)
+			(effects
+				(font
+					(size 1.27 1.27)
+				)
+			)
+		)
+		(property "Value" "22"
+			(at 158.496 95.504 90)
+			(effects
+				(font
+					(size 1.27 1.27)
+				)
+			)
+		)
+		(property "Footprint" "Resistor_SMD:R_0402_1005Metric_Pad0.72x0.64mm_HandSolder"
+			(at 158.75 91.948 90)
+			(effects
+				(font
+					(size 1.27 1.27)
+				)
+				(hide yes)
+			)
+		)
+		(property "Datasheet" "~"
+			(at 158.75 90.17 0)
+			(effects
+				(font
+					(size 1.27 1.27)
+				)
+				(hide yes)
+			)
+		)
+		(property "Description" "Resistor"
+			(at 158.75 90.17 0)
+			(effects
+				(font
+					(size 1.27 1.27)
+				)
+				(hide yes)
+			)
+		)
+		(pin "2"
+		)
+		(pin "1"
+		)
+		(instances
+			(project "60_keyboard"
+				(path "/60f4ab9d-718b-428d-904c-5042759d3860/a5dc5d45-cfa6-4235-a666-1339e0663470"
+					(reference "R8")
+					(unit 1)
+				)

Commit message: Finished board, with maybe some cleanup needed
Parts:
- L2: value 2n -> 24n
Connections:
- net +3.3V: now also C3.1, C4.1, U1.28 (VDDPST2), U1.5 (VDDPST1)
- net Col 1: now also U1.6 (GPIO0/XTAL_32K_P)
- net Col 10: now also U1.17 (GPIO11)
- net Col 11: now also U1.27 (GPIO15)
- net Col 12: now also U1.29 (U0TXD/GPIO16)
- net Col 2: now also U1.7 (GPIO1/XTAL_32K_N)
- net Col 3: now also U1.8 (GPIO2)
- net Col 4: now also U1.9 (GPIO3)
- net Col 5: now also U1.10 (GPIO4/MTMS)
- net Col 6: now also U1.11 (GPIO5/MTDI)
- net Col 7: now also U1.12 (GPIO6/MTCK)
- net Col 8: now also U1.13 (GPIO7/MTDO)
- net Col 9: now also U1.16 (GPIO10)
- net Row 1: now also U1.32 (SDIO_CLK/GPIO19)
- net Row 2: now also U1.33 (SDIO_DATA0/GPIO20)
- net Row 3: now also U1.34 (SDIO_DATA1/GPIO21)
- net Row 4: now also U1.35 (SDIO_DATA2/GPIO22)
- net Row 5: now also U1.36 (SDIO_DATA3/GPIO23)

Commit message: Creeated all fabrication outputs and such, but assembly is expensive when it is both sides. So I will look to  fix this.
Parts:
- C10, C11, C12, C14, C15, C3, C4, C5, C6, C7, C8, C9: footprint Resistor_SMD:R_0402_1005Metric_Pad0.72x0.64mm_HandSolder -> Capacitor_SMD:C_0402_1005Metric_Pad0.74x0.62mm_HandSolder
Changed lines of the file:
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@@
 			)
 		)
-		(property "Footprint" "Resistor_SMD:R_0402_1005Metric_Pad0.72x0.64mm_HandSolder"
+		(property "Footprint" "Capacitor_SMD:C_0402_1005Metric_Pad0.74x0.62mm_HandSolder"
 			(at 176.2252 80.01 0)
 			(effects
@@
 			)
 		)
-		(property "Footprint" "Resistor_SMD:R_0402_1005Metric_Pad0.72x0.64mm_HandSolder"
+		(property "Footprint" "Capacitor_SMD:C_0402_1005Metric_Pad0.74x0.62mm_HandSolder"
 			(at 234.6452 69.85 0)
 			(effects
@@
 			)
 		)
-		(property "Footprint" "Resistor_SMD:R_0402_1005Metric_Pad0.72x0.64mm_HandSolder"
+		(property "Footprint" "Capacitor_SMD:C_0402_1005Metric_Pad0.74x0.62mm_HandSolder"
 			(at 153.3652 82.55 0)
 			(effects
@@
 			)
 		)
-		(property "Footprint" "Resistor_SMD:R_0402_1005Metric_Pad0.72x0.64mm_HandSolder"
+		(property "Footprint" "Capacitor_SMD:C_0402_1005Metric_Pad0.74x0.62mm_HandSolder"
 			(at 260.0452 69.85 0)
 			(effects
@@
 			)
 		)
-		(property "Footprint" "Resistor_SMD:R_0402_1005Metric_Pad0.72x0.64mm_HandSolder"
+		(property "Footprint" "Capacitor_SMD:C_0402_1005Metric_Pad0.74x0.62mm_HandSolder"
 			(at 214.3252 74.93 0)
 			(effects
@@
 			)
 		)
-		(property "Footprint" "Resistor_SMD:R_0402_1005Metric_Pad0.72x0.64mm_HandSolder"
+		(property "Footprint" "Capacitor_SMD:C_0402_1005Metric_Pad0.74x0.62mm_HandSolder"
 			(at 271.4752 69.85 0)
 			(effects
@@
 			)
 		)
-		(property "Footprint" "Resistor_SMD:R_0402_1005Metric_Pad0.72x0.64mm_HandSolder"
+		(property "Footprint" "Capacitor_SMD:C_0402_1005Metric_Pad0.74x0.62mm_HandSolder"
 			(at 225.7552 74.93 0)
 			(effects
@@
 			)
 		)
-		(property "Footprint" "Resistor_SMD:R_0402_1005Metric_Pad0.72x0.64mm_HandSolder"
+		(property "Footprint" "Capacitor_SMD:C_0402_1005Metric_Pad0.74x0.62mm_HandSolder"
 			(at 187.6552 80.01 0)
 			(effects
@@
 			)
 		)
-		(property "Footprint" "Resistor_SMD:R_0402_1005Metric_Pad0.72x0.64mm_HandSolder"
+		(property "Footprint" "Capacitor_SMD:C_0402_1005Metric_Pad0.74x0.62mm_HandSolder"
 			(at 121.6152 172.72 0)
 			(effects
@@
 			)
 		)
-		(property "Footprint" "Resistor_SMD:R_0402_1005Metric_Pad0.72x0.64mm_HandSolder"
+		(property "Footprint" "Capacitor_SMD:C_0402_1005Metric_Pad0.74x0.62mm_HandSolder"
 			(at 164.7952 82.55 0)
 			(effects
@@
 			)
 		)
-		(property "Footprint" "Resistor_SMD:R_0402_1005Metric_Pad0.72x0.64mm_HandSolder"
+		(property "Footprint" "Capacitor_SMD:C_0402_1005Metric_Pad0.74x0.62mm_HandSolder"
 			(at 84.7852 172.72 0)
 			(effects
@@
 			)
 		)
-		(property "Footprint" "Resistor_SMD:R_0402_1005Metric_Pad0.72x0.64mm_HandSolder"
+		(property "Footprint" "Capacitor_SMD:C_0402_1005Metric_Pad0.74x0.62mm_HandSolder"
 			(at 247.3452 69.85 0)
 			(effects
